Commit message: Updated urdf

File: russell_fireworks_description/urdf/russell_fireworks_description.urdf.xacro (robot description, xacro)
@@ -3,3 +3,35 @@
   <xacro:include filename="$(find kuka_kr10_support)/urdf/kr10r1100sixx_macro.xacro" />
   <xacro:kuka_kr10r1100sixx prefix=""/>
+  <link name="russell_eoat_link">
+    <visual>
+      <origin xyz="0 0 0" rpy="0 0 0"/>
+      <geometry>
+          <mesh filename="package://russell_fireworks_description/meshes/EOAT_Simple.stl" />
+      </geometry>
+      <material name="zed2i_mat"/>
+    </visual>
+    <collision>
+      <origin xyz="0 0 0" rpy="0 0 0"/>
+      <geometry>
+          <mesh filename="package://russell_fireworks_description/meshes/EOAT_Simple.stl" />
+      </geometry>
+    </collision>
+  </link>
+  <joint name="russell_eoat_joint" type="fixed">
+    <parent link="tool0"/>
+    <child link="russell_eoat_link"/>
+    <origin xyz="0 0 0" rpy="0 0 0"/>
+  </joint>
+  <joint name="zed_link" type="fixed">
+    <parent link="russell_eoat_link"/>
+    <child link="zed_mount_link"/>
+    <origin xyz="0.042516 -0.017 0.0482" rpy="0 0 3.14159"/>
+  </joint>
+  <link name="zed_mount_link" />
+  <joint name="zed_joint" type="fixed">
+    <parent link="zed_mount_link" />
+    <child link="zed_link" />
+    <origin xyz="0 0 0.015" rpy="0 0 0"/>
+  </joint>
+  <xacro:include filename="$(find zed_interfaces)/urdf/zed2i_descr.urdf.xacro"/>
 </robot>

Commit message: Added tcp

File: russell_fireworks_description/urdf/russell_fireworks_description.urdf.xacro (robot description, xacro)
@@ -34,4 +34,10 @@
     <origin xyz="0 0 0.015" rpy="0 0 0"/>
   </joint>
+  <link name="hot_tcp_link" />
+  <joint name="hot_joint" type="fixed">
+    <parent link="russell_eoat_link" />
+    <child link="hot_tcp_link" />
+    <origin xyz="-0.1381 -0.017 0.0256" rpy="0 1.5708 3.14159"/>
+  </joint>
   <xacro:include filename="$(find russell_fireworks_description)/urdf/zed2i_descr.urdf.xacro"/>
 </robot>

Commit message: Added the platform  Fixed zed transparency

File: russell_fireworks_description/urdf/russell_fireworks_description.urdf.xacro (robot description, xacro)
@@ -3,4 +3,24 @@
   <xacro:include filename="$(find kuka_kr10_support)/urdf/kr10r1100sixx_macro.xacro" />
   <xacro:kuka_kr10r1100sixx prefix=""/>
+  <link name="platform_link">
+    <visual>
+      <origin xyz="0 0 0" rpy="0 0 0"/>
+      <geometry>
+          <mesh filename="package://russell_fireworks_description/meshes/Platform.stl" />
+      </geometry>
+      <material name="zed2i_mat"/>
+    </visual>
+    <collision>
+      <origin xyz="0 0 0" rpy="0 0 0"/>
+      <geometry>
+          <mesh filename="package://russell_fireworks_description/meshes/Platform.stl" />
+      </geometry>
+    </collision>
+  </link>
+  <joint name="platform_joint" type="fixed">
+    <parent link="base_link"/>
+    <child link="platform_link"/>
+    <origin xyz="0 0 0" rpy="0 0 0"/>
+  </joint>
   <link name="russell_eoat_link">
     <visual>
